File: ErgoDOX pcb/matrixcogs/protoMxCog/ErgoDOX.sch (KiCad schematic (older format))
At the start: 52 parts, among them J1 Conn_01x18, SW0:10 SW0:3, SW0:11 SW0:2, SW0:12 SW0:1, SW0:7 SW0:6, SW0:8 SW0:5, SW0:9 SW0:4, SW1:10 SW1:3, SW1:11 SW1:2, SW1:12 SW1:1, SW1:13 SW1:0, SW1:9 SW1:4, SW2:10 SW2:3, SW2:11 SW2:2, SW2:12 SW2:1, SW2:13 SW2:0, SW2:7 SW2:6, SW2:8 SW2:5, SW2:9 SW2:4, SW3:10 SW3:3, SW3:11 SW3:2, SW3:12 SW3:1, SW3:13 SW3:0, SW3:8 SW3:5, SW3:9 SW3:4, SW4:10 SW4:3, SW4:11 SW4:2, SW4:12 SW4:1, SW4:13 SW4:0, SW4:7 SW4:6, SW4:8 SW4:5, SW4:9 SW4:4, SW5:10 SW5:3, SW5:11 SW5:2, SW5:12 SW5:1, SW5:13 SW5:0, SW5:7 SW5:6, SW5:8 SW5:5, SW5:9 SW5:4

Commit message: removing top part of PCB on switch matrix board
Parts:
- D1:7, D1:8: footprint (none) -> ergodox:DIODE
- H99: footprint (none) -> ergodox:ErgoDOXmech
- J1: footprint (none) -> ergodox:ErgoCogs_side_con
- LED_A1, LED_B1: footprint (none) -> LED_SMD:LED_0805_2012Metric_Pad1.15x1.40mm_HandSolder
- R1, R2: footprint (none) -> Resistor_SMD:R_0603_1608Metric_Pad0.98x0.95mm_HandSolder
- S1, S2: footprint (none) -> ergodox:STAB_PCB940
- SW0:10, SW0:11, SW0:12, SW0:7, SW0:8, SW0:9, SW1:10, SW1:11, SW1:12, SW1:13, SW1:9, SW2:10, SW2:11, SW2:12, SW2:13, SW2:7, SW2:8, SW2:9, SW3:10, SW3:11, SW3:12, SW3:13, SW3:8, SW3:9, SW4:10, SW4:11, SW4:12, SW4:13, SW4:7, SW4:8, SW4:9, SW5:10, SW5:11, SW5:12, SW5:13, SW5:7, SW5:8, SW5:9, SX0:10, SX0:11, SX1:7, SX1:8: footprint (none) -> ergodox:MX_FLIP_DIODE

Commit message: refactoring library structure, finishing basic matrix cog
Parts:
- removed J1: Conn_01x18, ergodox:ErgoCogs_side_con, symbol Connector_Generic:Conn_01x18
- removed LED_A1: LEDa, LED_SMD:LED_0805_2012Metric_Pad1.15x1.40mm_HandSolder, symbol component:LED
- added D1, D4: WS2812B, LED_SMD:LED_WS2812B_PLCC4_5.0x5.0mm_P3.2mm, symbol LED:WS2812B
- added D2, D3: LED_R, LED_SMD:LED_0805_2012Metric_Pad1.15x1.40mm_HandSolder, symbol ergodox_components:LED
- added D6: LED_G, LED_SMD:LED_0805_2012Metric_Pad1.15x1.40mm_HandSolder, symbol ergodox_components:LED
- added J1: Conn_01x06, ergodox:ErgoCogs_sidecon_top, symbol Connector_Generic:Conn_01x06
- added J2: Conn_01x10, ergodox:ErgoCogs_sidecon_bot, symbol Connector_Generic:Conn_01x10
- added R3, R4: 470, Resistor_SMD:R_0603_1608Metric_Pad0.98x0.95mm_HandSolder, symbol Device:R_Small
- D1:7, D1:8: symbol component:DIODE -> ergodox_components:DIODE
- D5: renamed from LED_B1; value LEDb -> LED_G; symbol component:LED -> ergodox_components:LED
- H99, S1, S2: symbol component:ANYTHING -> ergodox_components:ANYTHING
- SW0:10, SW0:11, SW0:12, SW0:7, SW0:8, SW0:9, SW1:10, SW1:11, SW1:12, SW1:13, SW1:9, SW2:10, SW2:11, SW2:12, SW2:13, SW2:7, SW2:8, SW2:9, SW3:10, SW3:11, SW3:12, SW3:13, SW3:8, SW3:9, SW4:10, SW4:11, SW4:12, SW4:13, SW4:7, SW4:8, SW4:9, SW5:10, SW5:11, SW5:12, SW5:13, SW5:7, SW5:8, SW5:9: symbol component:SWITCH_DIODE -> ergodox_components:SWITCH_DIODE
- SX0:10, SX0:11, SX1:7, SX1:8: footprint ergodox:MX_FLIP_DIODE -> ergodox:MX_FLIP; symbol component:SWITCH_PUSH -> ergodox_components:SWITCH_PUSH
Connections:
- net LED_B is gone; now on net VCC: R1.1
- net COL0: now also J2.10 (Pin_10)
- net COL1: now also J2.9 (Pin_9)
- net COL10: now also J2.7 (Pin_7)
- net COL11: now also J2.8 (Pin_8)
- net COL4: now also J2.6 (Pin_6)
- net COL5: now also J2.5 (Pin_5)
- net COL6: now also J2.4 (Pin_4)
- net GND: now also D1.3 (VSS), D2.2 (K), D3.2 (K), D4.3 (VSS), D6.2 (K), J2.3 (Pin_3); no longer H99.0 (GND), S1.0 (GND), S2.0 (GND), SX0:10.0 (GND), SX0:11.0 (GND), SX1:7.0 (GND), SX1:8.0 (GND)
- net ROW0: now also J1.1 (Pin_1)
- net ROW1: now also J1.2 (Pin_2)
- net ROW2: now also J1.3 (Pin_3)
- net ROW3: now also J1.4 (Pin_4)
- net ROW4: now also J1.5 (Pin_5)
- net ROW5: now also J1.6 (Pin_6)
- net VCC: now also D1.1 (VDD), D4.1 (VDD), J2.1 (Pin_1), R3.1
- net at R1.2: now also D2.1 (A)
- net LED_A renamed LED_GPIO
- net LED_GPIO: now also D1.4 (DIN), D4.4 (DIN), J2.2 (Pin_2), R4.1
- new net: D6.1 (A), R4.2
- new net: D3.1 (A), R3.2
Other:
- note added: "BOT"
- note added: "TOP"
- moved on the sheet: D1:7, D1:8, D5, H99, R2, S1, S2, SW0:10, SW0:11, SW0:12, SW0:7, SW0:8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
