File: ErgoDOX pcb/matrixcogs/protoMxCog/protoMxCog.kicad_pcb (KiCad board)
At the start: 2 copper layers, 182.8 x 140.1 mm, 59 parts, among them J1 Conn_01x06, J2 Conn_01x10, SW0:10 SW0:3, SW0:11 SW0:2, SW0:12 SW0:1, SW0:7 SW0:6, SW0:8 SW0:5, SW0:9 SW0:4, SW1:10 SW1:3, SW1:11 SW1:2, SW1:12 SW1:1, SW1:13 SW1:0, SW1:9 SW1:4, SW2:10 SW2:3, SW2:11 SW2:2, SW2:12 SW2:1, SW2:13 SW2:0, SW2:7 SW2:6, SW2:8 SW2:5, SW2:9 SW2:4, SW3:10 SW3:3, SW3:11 SW3:2, SW3:12 SW3:1, SW3:13 SW3:0, SW3:8 SW3:5, SW3:9 SW3:4, SW4:10 SW4:3, SW4:11 SW4:2, SW4:12 SW4:1, SW4:13 SW4:0, SW4:7 SW4:6, SW4:8 SW4:5, SW4:9 SW4:4, SW5:10 SW5:3, SW5:11 SW5:2, SW5:12 SW5:1, SW5:13 SW5:0, SW5:7 SW5:6, SW5:8 SW5:5, SW5:9 SW5:4

Commit message: 1st version of braincogs
Parts:
- moved J1 6.00 mm to (74.5, 74.2)
- moved J2 6.00 mm to (74.6, 98.0)
Connections:
- net /COL0 renamed /COL0_13
- net /COL1 renamed /COL1_12
- net /COL10 renamed /COL3_10
- net /COL11 renamed /COL2_11
- net /COL4 renamed /COL4_9
- net /COL5 renamed /COL5_8
- net /COL6 renamed /COL6_7
Routing:
- net GND: track 11.5 -> 24.4 mm
- net VCC: track 166.3 -> 172.3 mm
- net /ROW5: track 209.6 -> 215.6 mm
- net /ROW3: track 193.8 -> 199.8 mm
- net /ROW2: track 219.9 -> 225.9 mm
- net /ROW1: track 283.2 -> 289.2 mm
- net /ROW0: track 308.4 -> 314.4 mm
- net /COL5_8: track 152.2 -> 158.2 mm
- net /COL3_10: track 205.3 -> 211.3 mm
- net /ROW4: track 168.8 -> 174.7 mm
- net /COL0_13: track 223.8 -> 228.9 mm
- net /COL1_12: track 299.5 -> 304.3 mm
- net /LED_GPIO: track 169.0 -> 173.7 mm
- net /COL2_11: track 299.1 -> 303.6 mm
- net /COL6_7: track 217.7 -> 221.5 mm
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Other:
- outline, holes or cut-outs redrawn
- board text removed: "Components are intended to be placed on the side they are drawn. It is however possible to invert the design. See the webpage for further instructions. www.ergodox.io"
