File: ErgoDOX pcb/matrixcogs/protoMxCog/protoMxCog.sch (KiCad schematic (older format))
At the start: 59 parts, among them J1 Conn_01x06, J2 Conn_01x10, SW0:10 SW0:3, SW0:11 SW0:2, SW0:12 SW0:1, SW0:7 SW0:6, SW0:8 SW0:5, SW0:9 SW0:4, SW1:10 SW1:3, SW1:11 SW1:2, SW1:12 SW1:1, SW1:13 SW1:0, SW1:9 SW1:4, SW2:10 SW2:3, SW2:11 SW2:2, SW2:12 SW2:1, SW2:13 SW2:0, SW2:7 SW2:6, SW2:8 SW2:5, SW2:9 SW2:4, SW3:10 SW3:3, SW3:11 SW3:2, SW3:12 SW3:1, SW3:13 SW3:0, SW3:8 SW3:5, SW3:9 SW3:4, SW4:10 SW4:3, SW4:11 SW4:2, SW4:12 SW4:1, SW4:13 SW4:0, SW4:7 SW4:6, SW4:8 SW4:5, SW4:9 SW4:4, SW5:10 SW5:3, SW5:11 SW5:2, SW5:12 SW5:1, SW5:13 SW5:0, SW5:7 SW5:6, SW5:8 SW5:5, SW5:9 SW5:4

Commit message: 1st version of braincogs
Connections:
- net labels added: COL0_13, COL1_12, COL2_11, COL3_10, COL4_9, COL5_8, COL6_7
- net labels removed: COL0, COL1, COL10, COL11, COL12, COL13, COL2, COL3, COL4, COL5, COL6, COL7, COL8, COL9
Changed lines of the file:
@@
 Text Label 5450 4900 2    60   ~ 0
 ROW0
-Text Label 6550 5700 3    60   ~ 0
-COL5
-Text Label 10050 5700 3    60   ~ 0
-COL0
-Text Label 9350 5700 3    60   ~ 0
-COL1
-Text Label 8650 5700 3    60   ~ 0
-COL2
-Text Label 7950 5700 3    60   ~ 0
-COL3
-Text Label 7250 5700 3    60   ~ 0
-COL4
+Text Label 9350 5650 3    60   ~ 0
+COL1_12
+Text Label 7250 5600 3    60   ~ 0
+COL4_9
 $Comp
 L ergodox_components:SWITCH_DIODE SW0:9
@@
 	1    0    0    -1
 $EndComp
-Text Label 9350 5400 3    60   ~ 0
-COL12
-Text Label 6550 5400 3    60   ~ 0
-COL8
-Text Label 10050 5400 3    60   ~ 0
-COL13
-Text Label 8650 5400 3    60   ~ 0
-COL11
-Text Label 7950 5400 3    60   ~ 0
-COL10
-Text Label 7250 5400 3    60   ~ 0
-COL9
+Text Label 8650 5600 3    60   ~ 0
+COL2_11
+Text Label 7950 5600 3    60   ~ 0
+COL3_10
 Wire Wire Line
 	6350 5250 6350 5150
@@
 	1    0    0    -1
 $EndComp
-Text Label 1450 2950 0    60   ~ 0
-COL6
-Text Label 1450 3050 0    60   ~ 0
-COL5
-Text Label 1450 3550 0    60   ~ 0
-COL0
-Text Label 1450 3450 0    60   ~ 0
-COL1
-Text Label 1450 3350 0    60   ~ 0
-COL2
-Text Label 1450 3250 0    60   ~ 0
-COL3
-Text Label 1450 3150 0    60   ~ 0
-COL4
-Text Label 1150 3450 0    60   ~ 0
-COL12
-Text Label 1150 2950 0    60   ~ 0
-COL7
+Text Label 1150 3550 0    60   ~ 0
+COL0_13
 Text Label 1150 3050 0    60   ~ 0
-COL8
-Text Label 1150 3550 0    60   ~ 0
-COL13
-Text Label 1150 3350 0    60   ~ 0
-COL11
-Text Label 1150 3250 0    60   ~ 0
-COL10
-Text Label 1150 3150 0    60   ~ 0
-COL9
+COL5_8
 Wire Wire Line
 	1000 2950 1450 2950
@@
 Wire Wire Line
 	1200 2150 1200 2650
-Text Label 5850 5400 3    60   ~ 0
-COL7
-Text Label 5850 5700 3    60   ~ 0
-COL6
 $Comp
 L ergodox_components:LED D2
@@
 Text Notes 4100 3700 0    50   ~ 0
 BOT
+Text Label 1150 2950 0    60   ~ 0
+COL6_7
+Text Label 5850 5550 3    60   ~ 0
+COL6_7
+Text Label 6550 5600 3    60   ~ 0
+COL5_8
+Text Label 1150 3450 0    60   ~ 0
+COL1_12
+Text Label 1150 3350 0    60   ~ 0
+COL2_11
+Text Label 1150 3250 0    60   ~ 0
+COL3_10
+Text Label 1150 3150 0    60   ~ 0
+COL4_9
+Text Label 10050 5600 3    60   ~ 0
+COL0_13
 $EndSCHEMATC
