File: ErgoDOX pcb/braincogs/protoSmortCog/protoSmortCog.sch (KiCad schematic (older format))
At the start: 64 parts, among them J1 USB, J2 3.5mm, J3 JMP, J4 JMP, SW0:10 SW0:3, SW0:11 SW0:2, SW0:12 SW0:1, SW0:7 SW0:6, SW0:8 SW0:5, SW0:9 SW0:4, SW1:10 SW1:3, SW1:11 SW1:2, SW1:12 SW1:1, SW1:13 SW1:0, SW1:9 SW1:4, SW2:10 SW2:3, SW2:11 SW2:2, SW2:12 SW2:1, SW2:13 SW2:0, SW2:7 SW2:6, SW2:8 SW2:5, SW2:9 SW2:4, SW3:10 SW3:3, SW3:11 SW3:2, SW3:12 SW3:1, SW3:13 SW3:0, SW3:8 SW3:5, SW3:9 SW3:4, SW4:10 SW4:3, SW4:11 SW4:2, SW4:12 SW4:1, SW4:13 SW4:0, SW4:7 SW4:6, SW4:8 SW4:5, SW4:9 SW4:4, SW5:10 SW5:3, SW5:11 SW5:2, SW5:12 SW5:1, SW5:13 SW5:0, SW5:7 SW5:6, SW5:8 SW5:5, SW5:9 SW5:4, U1 TEENSY2.0, U2 MCP23018

Commit message: adjusting former ergodox project for a smart cog template (WIP)
Parts:
- removed D1:7, D1:8: D, symbol component:DIODE
- removed H99: MECHANICAL, symbol component:ANYTHING
- removed J1: USB, symbol component:6PIN
- removed J2: 3.5mm, symbol component:6PIN
- removed J3, J4: JMP, symbol component:3PIN
- removed JP1, JP2: JUMPER, symbol component:JUMPER
- removed LED_A1: LEDa, symbol component:LED
- removed LED_B1: LEDb, symbol component:LED
- removed LED_C1: LEDc, symbol component:LED
- removed R1, R2: 2.2kΩ, symbol component:RESISTOR
- removed RA1: LEDa, symbol component:RESISTOR
- removed RB1: LEDb, symbol component:RESISTOR
- removed RC1: LEDc, symbol component:RESISTOR
- removed S1, S2: STAB200, symbol component:ANYTHING
- removed SW0:10: SW0:3, symbol component:SWITCH_DIODE
- removed SW0:11: SW0:2, symbol component:SWITCH_DIODE
- removed SW0:12: SW0:1, symbol component:SWITCH_DIODE
- removed SW0:7: SW0:6, symbol component:SWITCH_DIODE
- removed SW0:8: SW0:5, symbol component:SWITCH_DIODE
- removed SW0:9: SW0:4, symbol component:SWITCH_DIODE
- removed SW1:10: SW1:3, symbol component:SWITCH_DIODE
- removed SW1:11: SW1:2, symbol component:SWITCH_DIODE
- removed SW1:12: SW1:1, symbol component:SWITCH_DIODE
- removed SW1:13: SW1:0, symbol component:SWITCH_DIODE
- removed SW1:9: SW1:4, symbol component:SWITCH_DIODE
- removed SW2:10: SW2:3, symbol component:SWITCH_DIODE
- removed SW2:11: SW2:2, symbol component:SWITCH_DIODE
- removed SW2:12: SW2:1, symbol component:SWITCH_DIODE
- removed SW2:13: SW2:0, symbol component:SWITCH_DIODE
- removed SW2:7: SW2:6, symbol component:SWITCH_DIODE
- removed SW2:8: SW2:5, symbol component:SWITCH_DIODE
- removed SW2:9: SW2:4, symbol component:SWITCH_DIODE
- removed SW3:10: SW3:3, symbol component:SWITCH_DIODE
- removed SW3:11: SW3:2, symbol component:SWITCH_DIODE
- removed SW3:12: SW3:1, symbol component:SWITCH_DIODE
- removed SW3:13: SW3:0, symbol component:SWITCH_DIODE
- removed SW3:8: SW3:5, symbol component:SWITCH_DIODE
- removed SW3:9: SW3:4, symbol component:SWITCH_DIODE
- removed SW4:10: SW4:3, symbol component:SWITCH_DIODE
- removed SW4:11: SW4:2, symbol component:SWITCH_DIODE
- removed SW4:12: SW4:1, symbol component:SWITCH_DIODE
- removed SW4:13: SW4:0, symbol component:SWITCH_DIODE
- removed SW4:7: SW4:6, symbol component:SWITCH_DIODE
- removed SW4:8: SW4:5, symbol component:SWITCH_DIODE
- removed SW4:9: SW4:4, symbol component:SWITCH_DIODE
- removed SW5:10: SW5:3, symbol component:SWITCH_DIODE
- removed SW5:11: SW5:2, symbol component:SWITCH_DIODE
- removed SW5:12: SW5:1, symbol component:SWITCH_DIODE
- removed SW5:13: SW5:0, symbol component:SWITCH_DIODE
- removed SW5:7: SW5:6, symbol component:SWITCH_DIODE
- removed SW5:8: SW5:5, symbol component:SWITCH_DIODE
- removed SW5:9: SW5:4, symbol component:SWITCH_DIODE
- removed SX0:10: SX0:3, symbol component:SWITCH_PUSH
- removed SX0:11: SX0:2, symbol component:SWITCH_PUSH
- removed SX1:7: SX1:6, symbol component:SWITCH_PUSH
- removed SX1:8: SX1:5, symbol component:SWITCH_PUSH
- removed U2: MCP23018, symbol component:MCP23018
- added D1, D2, D3: LED, LED_THT:LED_D3.0mm_Clear, symbol Device:LED
- added J1: AudioJack4_SwitchTR1, Connector_Audio:Jack_3.5mm_PJ311_Horizontal, symbol Connector:AudioJack4_SwitchTR1
- added J2: USB_C_Receptacle_USB2.0, Connector_USB:USB_C_Receptacle_GCT_USB4085, symbol Connector:USB_C_Receptacle_USB2.0
- added J5: Conn_01x06, ergodox:ErgoCogs_sidecon_top, symbol Connector_Generic:Conn_01x06
- added J6: Conn_01x10, ergodox:ErgoCogs_sidecon_bot, symbol Connector_Generic:Conn_01x10
- added R1, R2, R3, R4, R5, R6, R7: 4k7, Resistor_SMD:R_0603_1608Metric_Pad0.98x0.95mm_HandSolder, symbol Device:R_Small
- added U2: MCP23017_SO, Package_SO:SOIC-28W_7.5x17.9mm_P1.27mm, symbol Interface_Expansion:MCP23017_SO
- SW_RST1: footprint Buttons_Switches_SMD:SW_SPST_B3U-1000P -> Button_Switch_SMD:SW_SPST_TL3342; symbol component:SWITCH_PUSH -> ergodox_components:SWITCH_PUSH
- U1: footprint (none) -> ergodox:TEENSY_2.0_WITH_RESET; symbol component:TEENSY2.0 -> ergodox_components:TEENSY2.0
Connections:
- net labels added: LED_GPIO, SCL, SDA, VBUS
- net labels removed: SCLM, SCLS, SDAM, SDAS
- wire segments 253 -> 91
- no-connect marks 15 -> 16
