File: ErgoDOX pcb/braincogs/alphaBrain/alphaRightHemi/alphaRightHemi.kicad_pcb (KiCad board)
At the start: 2 copper layers, 37 x 86 mm, 14 parts, among them J1 AudioJack4, J2 USB_C_Receptacle_USB2.0, J5 Conn_01x06, J6 Conn_01x10, U1 TEENSY2.0

Commit message: repo cleanup, adding fab files for PCBs
Other:
- board text added: "ErgoCogs alphaBrain rev. 1"
