File: ErgoDOX pcb/braincogs/alphaBrain/alphaLeftHemi/alphaLeftHemi.kicad_pcb (KiCad board)
At the start: 2 copper layers, 37 x 86 mm, 13 parts, among them J1 AudioJack4, J5 Conn_01x06, J6 Conn_01x10, U2 MCP23018

Commit message: repo cleanup, adding fab files for PCBs
Parts:
- D1, D2, J1: moved to B.Cu
- moved C1 10.8 mm to (140.2, 53.5), turned to 90 degrees
- moved R4 6.35 mm to (132.8, 67.7), turned to 270 degrees
- moved R5 4.29 mm to (131.2, 67.7), turned to 270 degrees
- turned J1 to 0 degrees
Routing:
- net VCC: track 80.9 -> 92.5 mm
- net GND: track 166.1 -> 158.8 mm
- net /SDA: track 41.4 -> 43.3 mm
- net /SCL: track 29.5 -> 28.2 mm
Other:
- board text added: "ErgoCogs alphaBrain rev. 1"
- board text added: "This side up"
